Commit message: gazebo

File: description/gazebo_control.xacro (robot description, xacro)
@@ -6,5 +6,5 @@
             <left_joint>left_wheel_joint</left_joint>
             <right_joint>right_wheel_joint</right_joint>
-            <wheel_seperation>0.4</wheel_seperation>
+            <wheel_seperation>0.632</wheel_seperation>
             <wheel_diameter>0.1</wheel_diameter>
             <!--LIMITS-->

File: description/robot_core.xacro (robot description, xacro)
@@ -48,5 +48,5 @@
         <parent link = "base_link"/>
         <child link = "left_wheel"/>
-        <origin xyz = "0 0.2 0" rpy = "-${pi/2} 0 0"/>
+        <origin xyz = "0 0.316 0" rpy = "-${pi/2} 0 0"/>
         <axis xyz = "0 0 1"/>
     </joint>
@@ -74,5 +74,5 @@
         <parent link = "base_link"/>
         <child link = "right_wheel"/>
-        <origin xyz = "0 -0.2 0" rpy = "${pi/2} 0 0"/>
+        <origin xyz = "0 -0.316 0" rpy = "${pi/2} 0 0"/>
         <axis xyz = "0 0 -1"/>
     </joint>
