Commit message: hm

File: description/lidar.xacro (robot description, xacro)
@@ -4,5 +4,5 @@
         <parent link = "chassis"/>
         <child link = "lidar_frame"/>
-        <origin xyz = "0 0 0.2" rpy = "0 0 0"/>
+        <origin xyz = "0 0 0.1" rpy = "0 0 0"/>
     </joint>
     <link name = "lidar_frame">

Commit message: LIDAR!

File: description/lidar.xacro (robot description, xacro)
@@ -4,5 +4,5 @@
         <parent link = "chassis"/>
         <child link = "lidar_frame"/>
-        <origin xyz = "0 0 0.1" rpy = "0 0 0"/>
+        <origin xyz = "0 0 0.05" rpy = "0 0 0"/>
     </joint>
     <link name = "lidar_frame">
@@ -11,5 +11,5 @@
                 <cylinder radius = "0.04" length = "0.04"/>
             </geometry>
-            <material name = "black"/>
+            <material name = "red"/>
         </visual>
         <collision>
@@ -22,3 +22,32 @@
         </xacro:inertial_cylinder>
     </link>
+    <!--GAZEBO STUFF-->
+    <gazebo reference="lidar_frame">
+        <material>Gazebo/Red</material>
+        <sensor name="lidar" type="ray">
+            <pose> 0 0 0 0 0 0 </pose>
+            <visualize>true</visualize>
+            <update_rate>10</update_rate>
+            <ray>
+                <scan>
+                    <horizontal>
+                        <samples>360</samples>
+                        <min_angle>-3.14</min_angle>
+                        <max_angle>3.14</max_angle>
+                    </horizontal>
+                </scan>
+                <range>
+                    <min>0.3</min>
+                    <max>12</max>
+                </range>
+            </ray>
+            <plugin name="lidar_controller" filename="libgazebo_ros_ray_sensor.so">
+                <ros>
+                    <argument>~/out:=scan</argument>
+                </ros>
+                <output_type>sensor_msgs/LaserScan</output_type>
+                <frame_name>lidar_frame</frame_name>
+            </plugin>
+        </sensor>
+    </gazebo>
 </robot>

File: description/robot_core.xacro (robot description, xacro)
@@ -13,4 +13,7 @@
     <material name="black">
         <color rgba="0 0 0 1" />
+    </material>
+    <material name="red">
+        <color rgba = "1 0 0 1"/>
     </material>
     <!-- BASE LINK-->

Commit message: lidar

File: description/lidar.xacro (robot description, xacro)
@@ -4,5 +4,5 @@
         <parent link = "chassis"/>
         <child link = "lidar_frame"/>
-        <origin xyz = "0 0 0.05" rpy = "0 0 0"/>
+        <origin xyz = "0 0 0.07" rpy = "0 0 0"/>
     </joint>
     <link name = "lidar_frame">

Commit message: LIDAR

File: description/lidar.xacro (robot description, xacro)
@@ -4,5 +4,5 @@
         <parent link = "chassis"/>
         <child link = "lidar_frame"/>
-        <origin xyz = "0 0 0.07" rpy = "0 0 0"/>
+        <origin xyz = "0 0 0.15" rpy = "0 0 0"/>
     </joint>
     <link name = "lidar_frame">

Commit message: lidar

File: description/lidar.xacro (robot description, xacro)
@@ -4,5 +4,5 @@
         <parent link = "chassis"/>
         <child link = "lidar_frame"/>
-        <origin xyz = "0 0 0.15" rpy = "0 0 0"/>
+        <origin xyz = "0 0 0.12" rpy = "0 0 0"/>
     </joint>
     <link name = "lidar_frame">

Commit message: laser_frame rename to work on rplidar node

File: description/lidar.xacro (robot description, xacro)
@@ -3,8 +3,8 @@
     <joint name = "lidar_joint" type="fixed">
         <parent link = "chassis"/>
-        <child link = "lidar_frame"/>
+        <child link = "laser_frame"/>
         <origin xyz = "0 0 0.12" rpy = "0 0 0"/>
     </joint>
-    <link name = "lidar_frame">
+    <link name = "laser_frame">
         <visual>
             <geometry>
@@ -23,5 +23,5 @@
     </link>
     <!--GAZEBO STUFF-->
-    <gazebo reference="lidar_frame">
+    <gazebo reference="laser_frame">
         <material>Gazebo/Red</material>
         <sensor name="lidar" type="gpu_lidar">
@@ -44,5 +44,5 @@
             <topic>scan</topic>
             <!--<output_type>sensor_msgs/LaserScan</output_type>-->
-            <gz_frame_id>lidar_frame</gz_frame_id>
+            <gz_frame_id>laser_frame</gz_frame_id>
         </sensor>
     </gazebo>
