Commit message: help

File: description/robot_core.xacro (robot description, xacro)
@@ -1,4 +1,5 @@
 <?xml version="1.0"?>
 <robot xmlns:xacro="http://www.ros.org/wiki/xacro" >
+    <xacro:include filename = "inertial_macros.xacro"/>
     <material name="white">
         <color rgba="1 1 1 1" />
@@ -30,4 +31,13 @@
             <material name="white"/>
         </visual>
+        <collision>
+            <origin xyz="0 0 0"/>
+            <geometry>
+                <cylinder radius = "0.3" length = "0.05"/>
+            </geometry>
+        </collision>
+        <xacro:inertial_cylinder mass = "0.5" length = "0.05" radius = "0.3">
+            <origin xyz = "0 0 0" rpy = "0 0 0"/>
+        </xacro:inertial_cylinder>
     </link>
     <!--LEFT WHEEL LINK-->
@@ -45,4 +55,12 @@
             <material name = "black"/>
         </visual>
+        <collision>
+            <geometry>
+                <cylinder radius = "0.1" length = "0.03"/>
+            </geometry>
+        </collision>
+        <xacro:inertial_cylinder mass = "0.1" length = "0.03" radius = "0.1">
+            <origin xyz = "0 0 0" rpy = "0 0 0"/>
+        </xacro:inertial_cylinder>
     </link>
     <!--RIGHT WHEEL LINK-->
@@ -60,4 +78,12 @@
             <material name = "black"/>
         </visual>
+        <collision>
+            <geometry>
+                <cylinder radius = "0.1" length = "0.03"/>
+            </geometry>
+        </collision>
+        <xacro:inertial_cylinder mass = "0.1" length = "0.03" radius = "0.1">
+            <origin xyz = "0 0 0" rpy = "0 0 0"/>
+        </xacro:inertial_cylinder>
     </link>
     <!--CASTER WHEEL1 LINK-->
@@ -74,4 +100,12 @@
             <material name = "black"/>
         </visual>
+         <collision>
+            <geometry>
+                <sphere radius = "0.035"/>
+            </geometry>
+        </collision>
+        <xacro:inertial_sphere mass = "0.1" radius = "0.035">
+            <origin xyz = "0 0 0" rpy = "0 0 0"/>
+        </xacro:inertial_sphere>
     </link>
     <!--CASTER WHEEL2 LINK-->
@@ -88,4 +122,12 @@
             <material name = "black"/>
         </visual>
+        <collision>
+            <geometry>
+                <sphere radius = "0.035"/>
+            </geometry>
+        </collision>
+        <xacro:inertial_sphere mass = "0.1" radius = "0.035">
+            <origin xyz = "0 0 0" rpy = "0 0 0"/>
+        </xacro:inertial_sphere>
     </link>
 </robot>

Commit message: Gazebo sim

File: description/robot_core.xacro (robot description, xacro)
@@ -41,4 +41,7 @@
         </xacro:inertial_cylinder>
     </link>
+    <gazebo reference = "chassis">
+        <material>Gazebo/White</material>
+    </gazebo>
     <!--LEFT WHEEL LINK-->
     <joint name="left_wheel joint" type = "continuous">
@@ -64,4 +67,7 @@
         </xacro:inertial_cylinder>
     </link>
+    <gazebo reference = "left_wheel">
+        <material>Gazebo/Black</material>
+    </gazebo>
     <!--RIGHT WHEEL LINK-->
     <joint name="right_wheel joint" type = "continuous">
@@ -87,4 +93,7 @@
         </xacro:inertial_cylinder>
     </link>
+    <gazebo reference = "right_wheel">
+        <material>Gazebo/Black</material>
+    </gazebo>
     <!--CASTER WHEEL1 LINK-->
     <joint name = "caster_wheel1_joint" type = "fixed">
@@ -109,4 +118,7 @@
         </xacro:inertial_sphere>
     </link>
+    <gazebo reference = "caster_wheel1">
+        <material>Gazebo/Gray</material>
+    </gazebo>
     <!--CASTER WHEEL2 LINK-->
     <joint name = "caster_wheel2_joint" type = "fixed">
@@ -131,3 +143,6 @@
         </xacro:inertial_sphere>
     </link>
+    <gazebo reference = "caster_wheel2">
+        <material>Gazebo/Gray</material>
+    </gazebo>
 </robot>

Commit message: gazebo

File: description/robot_core.xacro (robot description, xacro)
@@ -45,5 +45,5 @@
     </gazebo>
     <!--LEFT WHEEL LINK-->
-    <joint name="left_wheel joint" type = "continuous">
+    <joint name="left_wheel_joint" type = "continuous">
         <parent link = "base_link"/>
         <child link = "left_wheel"/>
@@ -71,5 +71,5 @@
     </gazebo>
     <!--RIGHT WHEEL LINK-->
-    <joint name="right_wheel joint" type = "continuous">
+    <joint name="right_wheel_joint" type = "continuous">
         <parent link = "base_link"/>
         <child link = "right_wheel"/>

Commit message: Gazebo & odometry

File: description/robot_core.xacro (robot description, xacro)
@@ -100,10 +100,10 @@
         <parent link = "chassis"/>
         <child link = "caster_wheel1"/>
-        <origin xyz = "0.25 0 -0.05"/>
+        <origin xyz = "0.25 0 -0.06"/>
     </joint>
     <link name = "caster_wheel1">
         <visual>
             <geometry>
-                <sphere radius = "0.035"/>
+                <sphere radius = "0.039"/>
             </geometry>
             <material name = "black"/>
@@ -111,8 +111,8 @@
          <collision>
             <geometry>
-                <sphere radius = "0.035"/>
+                <sphere radius = "0.039"/>
             </geometry>
         </collision>
-        <xacro:inertial_sphere mass = "0.1" radius = "0.035">
+        <xacro:inertial_sphere mass = "0.1" radius = "0.039">
             <origin xyz = "0 0 0" rpy = "0 0 0"/>
         </xacro:inertial_sphere>
@@ -120,4 +120,6 @@
     <gazebo reference = "caster_wheel1">
         <material>Gazebo/Gray</material>
+        <mu1 value = "0.001"/>
+        <mu2 value = "0.001"/>
     </gazebo>
     <!--CASTER WHEEL2 LINK-->
@@ -125,10 +127,10 @@
         <parent link = "chassis"/>
         <child link = "caster_wheel2"/>
-        <origin xyz = "-0.25 0 -0.05"/>
+        <origin xyz = "-0.25 0 -0.06"/>
     </joint>
     <link name = "caster_wheel2">
         <visual>
             <geometry>
-                <sphere radius = "0.035"/>
+                <sphere radius = "0.039"/>
             </geometry>
             <material name = "black"/>
@@ -136,8 +138,8 @@
         <collision>
             <geometry>
-                <sphere radius = "0.035"/>
+                <sphere radius = "0.039"/>
             </geometry>
         </collision>
-        <xacro:inertial_sphere mass = "0.1" radius = "0.035">
+        <xacro:inertial_sphere mass = "0.1" radius = "0.039">
             <origin xyz = "0 0 0" rpy = "0 0 0"/>
         </xacro:inertial_sphere>
@@ -145,4 +147,6 @@
     <gazebo reference = "caster_wheel2">
         <material>Gazebo/Gray</material>
+        <mu1 value = "0.001"/>
+        <mu2 value = "0.001"/>
     </gazebo>
 </robot>

Commit message: lidar

File: description/robot_core.xacro (robot description, xacro)
@@ -103,5 +103,5 @@
         <parent link = "chassis"/>
         <child link = "caster_wheel1"/>
-        <origin xyz = "0.25 0 -0.06"/>
+        <origin xyz = "0.25 0 -0.065"/>
     </joint>
     <link name = "caster_wheel1">
@@ -130,5 +130,5 @@
         <parent link = "chassis"/>
         <child link = "caster_wheel2"/>
-        <origin xyz = "-0.25 0 -0.06"/>
+        <origin xyz = "-0.25 0 -0.065"/>
     </joint>
     <link name = "caster_wheel2">

Commit message: lidar!!!

File: description/robot_core.xacro (robot description, xacro)
@@ -103,5 +103,5 @@
         <parent link = "chassis"/>
         <child link = "caster_wheel1"/>
-        <origin xyz = "0.25 0 -0.065"/>
+        <origin xyz = "0.25 0 -0.062"/>
     </joint>
     <link name = "caster_wheel1">
@@ -130,5 +130,5 @@
         <parent link = "chassis"/>
         <child link = "caster_wheel2"/>
-        <origin xyz = "-0.25 0 -0.065"/>
+        <origin xyz = "-0.25 0 -0.062"/>
     </joint>
     <link name = "caster_wheel2">

Commit message: e

File: description/robot_core.xacro (robot description, xacro)
@@ -103,5 +103,5 @@
         <parent link = "chassis"/>
         <child link = "caster_wheel1"/>
-        <origin xyz = "0.25 0 -0.062"/>
+        <origin xyz = "0.25 0 -0.06"/>
     </joint>
     <link name = "caster_wheel1">
@@ -130,5 +130,5 @@
         <parent link = "chassis"/>
         <child link = "caster_wheel2"/>
-        <origin xyz = "-0.25 0 -0.062"/>
+        <origin xyz = "-0.25 0 -0.06"/>
     </joint>
     <link name = "caster_wheel2">

Commit message: lidar

File: description/robot_core.xacro (robot description, xacro)
@@ -103,5 +103,5 @@
         <parent link = "chassis"/>
         <child link = "caster_wheel1"/>
-        <origin xyz = "0.25 0 -0.06"/>
+        <origin xyz = "0.25 0 -0.0605"/>
     </joint>
     <link name = "caster_wheel1">
@@ -130,5 +130,5 @@
         <parent link = "chassis"/>
         <child link = "caster_wheel2"/>
-        <origin xyz = "-0.25 0 -0.06"/>
+        <origin xyz = "-0.25 0 -0.0605"/>
     </joint>
     <link name = "caster_wheel2">

Commit message: e

File: description/robot_core.xacro (robot description, xacro)
@@ -24,5 +24,5 @@
         <parent link="base_link"/>
         <child link="chassis"/>
-        <origin xyz="0 0 0"/>
+        <origin xyz="0 0 0.1"/>
     </joint>
     <link name ="chassis">
@@ -51,5 +51,5 @@
         <parent link = "base_link"/>
         <child link = "left_wheel"/>
-        <origin xyz = "0 0.316 0" rpy = "-${pi/2} 0 0"/>
+        <origin xyz = "0 0.316 0.1" rpy = "-${pi/2} 0 0"/>
         <axis xyz = "0 0 1"/>
     </joint>
@@ -77,5 +77,5 @@
         <parent link = "base_link"/>
         <child link = "right_wheel"/>
-        <origin xyz = "0 -0.316 0" rpy = "${pi/2} 0 0"/>
+        <origin xyz = "0 -0.316 0.1" rpy = "${pi/2} 0 0"/>
         <axis xyz = "0 0 -1"/>
     </joint>

Commit message: help

File: description/robot_core.xacro (robot description, xacro)
@@ -24,5 +24,5 @@
         <parent link="base_link"/>
         <child link="chassis"/>
-        <origin xyz="0 0 0.1"/>
+        <origin xyz="0 0 0.12"/>
     </joint>
     <link name ="chassis">
@@ -51,5 +51,5 @@
         <parent link = "base_link"/>
         <child link = "left_wheel"/>
-        <origin xyz = "0 0.316 0.1" rpy = "-${pi/2} 0 0"/>
+        <origin xyz = "0 0.316 0.12" rpy = "-${pi/2} 0 0"/>
         <axis xyz = "0 0 1"/>
     </joint>
@@ -77,5 +77,5 @@
         <parent link = "base_link"/>
         <child link = "right_wheel"/>
-        <origin xyz = "0 -0.316 0.1" rpy = "${pi/2} 0 0"/>
+        <origin xyz = "0 -0.316 0.12" rpy = "${pi/2} 0 0"/>
         <axis xyz = "0 0 -1"/>
     </joint>
